File: buck2.sch (KiCad schematic (older format))
At the start: 22 parts, among them J1 436500400, M1 30V,56Amps, M2 30V,35Amps, U1 TPS40303DRCR

Commit message: More new
Changed lines of the file:
@@
 U 1 1 60AACC27
 P 2750 2100
-F 0 "Cvcc1" H 2635 2054 50  0001 R CNN
+F 0 "Cvcc1" H 2635 2054 50  0000 R CNN
 F 1 "1uF,1mOhm" H 2635 2145 50  0000 R CNN
 F 2 "Capacitor_SMD:C_0805_2012Metric" H 2788 1950 50  0001 C CNN
@@
 U 1 1 60AE00A4
 P 6300 2000
-F 0 "M1" V 6846 2128 50  0001 L CNN
+F 0 "M1" V 6846 2128 50  0000 L CNN
 F 1 "30V,56Amps" V 6755 2128 50  0000 L CNN
 F 2 "buck2_footprint_custom_library:DQG_VSON-CLIP" H 7150 2100 50  0001 L CNN
@@
 U 1 1 60B291E6
 P 3750 2050
-F 0 "Css1" V 3754 2153 50  0001 L CNN
+F 0 "Css1" V 3754 2153 50  0000 L CNN
 F 1 "3.3nF,1mOhm" V 3845 2153 50  0000 L CNN
 F 2 "CAPC0603X33N" H 3750 2050 50  0001 L BNN
