File: buck2.kicad_pcb (KiCad board)
At the start: 2 copper layers, 22 parts, among them J1 436500400, M1 30V,56Amps, M2 30V,35Amps, U1 TPS40303DRCR

Commit message: new
Parts:
- moved Cvcc1 229.4 mm to (53.3, 89.8), turned to 270 degrees
- moved U1 225.6 mm to (58.4, 88.9)
- moved Css1 218.2 mm to (55.9, 94.0), turned to 270 degrees
- moved Rpgood1 217.9 mm to (53.3, 80.5), turned to 90 degrees
- moved Cin2 216.1 mm to (54.6, 97.8)
- moved Rs1 214.1 mm to (66.0, 86.4), turned to 270 degrees
- moved J1 211.6 mm to (64.8, 102.9)
- moved Cout1 211.2 mm to (73.7, 110.5), turned to 90 degrees
- moved Cbyp1 210.0 mm to (53.3, 86.4), turned to 270 degrees
- moved Cin1 208.9 mm to (54.6, 94.0)
- moved Cbst1 208.0 mm to (63.0, 85.1), turned to 180 degrees
- moved M2 207.0 mm to (63.5, 94.0), turned to 270 degrees
- moved Rfbt1 205.7 mm to (71.1, 106.7), turned to 90 degrees
- moved Ccomp2 203.7 mm to (73.7, 86.4)
- moved Rcomp1 200.7 mm to (73.7, 88.9), turned to 270 degrees
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Other:
- board outline added: 52.1 x 30.5 mm

Commit message: more
Parts:
- moved Cvcc1 48.2 mm to (99.4, 104.1), turned to 180 degrees
- moved Cin1 47.9 mm to (99.1, 111.8)
- moved Cin2 45.6 mm to (99.1, 108.0)
- moved Css1 43.2 mm to (95.2, 111.8), turned to 90 degrees
- moved Cbst1 41.0 mm to (83.3, 120.7)
- moved Rpgood1 41.0 mm to (73.7, 116.1)
- moved U1 39.5 mm to (91.4, 110.5), turned to 180 degrees
- moved Cbyp1 36.1 mm to (81.3, 109.2), turned to 90 degrees
- moved Rs1 33.3 mm to (87.6, 111.8)
- moved Ccomp1 28.5 mm to (94.0, 102.9), turned to 270 degrees
- moved L1 26.7 mm to (63.5, 99.1), turned to 90 degrees
- moved M2 26.4 mm to (85.1, 109.2), turned to 90 degrees
- moved Ccomp2 24.3 mm to (90.2, 104.1), turned to 180 degrees
- moved J1 24.1 mm to (87.6, 95.2), turned to 180 degrees
- moved Cout1 23.7 mm to (80.0, 87.6), turned to 270 degrees
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Routing:
- net Vout1: track 0.00 -> 31.4 mm
- net Net-(Cbst1-Pad2): track 0.00 -> 18.0 mm
- net FB-1: track 0.00 -> 15.8 mm
- net Vin1: track 0.00 -> 13.8 mm
- net Net-(Ccomp1-Pad2): track 0.00 -> 9.52 mm
- net Net-(M1-Pad4): track 0.00 -> 6.88 mm
- net Net-(M2-Pad4): track 0.00 -> 4.07 mm
- net Net-(Ccomp1-Pad1): track 0.00 -> 3.62 mm
- net Net-(Css1-Pad1): track 0.00 -> 2.85 mm
- net Net-(Ccomp3-Pad1): track 0.00 -> 2.48 mm
- net Net-(Rpgood1-Pad1): track 0.00 -> 2.41 mm

Commit message: More new
Parts:
- moved Rpgood1 28.3 mm to (100.3, 106.7), turned to 0 degrees
- moved Cbst1 17.0 mm to (91.0, 105.4)
- moved Cbyp1 15.7 mm to (96.5, 113.0), turned to 0 degrees
- moved Rfbt1 13.5 mm to (80.0, 109.2)
- moved Rcomp2 13.1 mm to (76.2, 111.8)
- moved Ccomp3 12.9 mm to (80.5, 111.8)
- moved Rcomp1 12.5 mm to (85.1, 113.0)
- moved Cin1 12.0 mm to (92.7, 101.6), turned to 270 degrees
- moved Rfbb1 10.2 mm to (85.1, 111.8)
- moved Ccomp1 9.67 mm to (90.2, 111.8), turned to 90 degrees
- moved Ccomp2 8.13 mm to (85.1, 110.5)
- moved Cin2 6.84 mm to (96.5, 101.6), turned to 270 degrees
- moved Css1 6.35 mm to (100.3, 108.0), turned to 0 degrees
- moved U1 4.58 mm to (95.2, 108.0)
- moved Rs1 3.81 mm to (87.6, 108.0), turned to 90 degrees
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Routing:
- net Vin1: track 13.8 -> 41.4 mm
- net Vout1: track 31.4 -> 43.8 mm
- net Net-(Cbyp1-Pad1): track 0.00 -> 6.34 mm, vias 0 -> 2
- net Net-(Cbst1-Pad2): track 18.0 -> 21.9 mm, vias 0 -> 2
- net Net-(Cbst1-Pad1): track 0.00 -> 3.05 mm
- net Net-(M1-Pad4): track 6.88 -> 9.61 mm
- net Net-(M2-Pad4): track 4.07 -> 6.73 mm
- net Net-(Rpgood1-Pad1): track 2.41 -> 3.70 mm
- net Net-(Ccomp1-Pad1): track 3.62 -> 4.89 mm
- net Net-(Ccomp1-Pad2): track 9.52 -> 8.28 mm, vias 0 -> 1
- net Net-(Css1-Pad1): track 2.85 -> 3.61 mm
- net FB-1: track 15.8 -> 15.5 mm, vias 0 -> 2
Other:
- board size 52.1 x 30.5 mm -> 52.1 x 31.8 mm

Commit message: New
Routing:
- net Vin2: track 0.00 -> 7.03 mm
- net Net-(Cbst1-Pad2): track 21.9 -> 25.6 mm
- added copper zone on F.Cu, net Vin2

Commit message: New
Routing:
- net FB-1: track 15.5 -> 36.1 mm
- net Net-(Ccomp1-Pad2): track 8.28 -> 22.0 mm, vias 1 -> 2
- net Vin2: track 7.03 -> 18.4 mm
- net Net-(Cbyp1-Pad1): track 6.34 -> 15.0 mm
- net Net-(Cbst1-Pad2): track 25.6 -> 27.5 mm
- net Net-(M2-Pad4): track 6.73 -> 8.39 mm
- net Vin1: track 41.4 -> 42.4 mm
- net Vout1: track 43.8 -> 44.7 mm, vias 0 -> 2
Other:
- board size 52.1 x 31.8 mm -> 54 x 31.8 mm
